File: pcb/ergotonic_f24-pcb-left/ergotonic_f24-pcb-left.kicad_pcb (KiCad board)
At the start: 2 copper layers, 167.2 x 112.2 mm, 66 parts, among them J1 Conn_01x04, J3 Conn_01x06, SW1 SW_PUSH, SW10 SW_PUSH, SW11 SW_PUSH, SW12 SW_PUSH, SW13 SW_PUSH, SW14 SW_PUSH, SW15 SW_PUSH, SW16 SW_PUSH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

Commit message: Version 1 Revision 3
Connections:
- J3 pad 6: unconnected-(J3-Pad6) -> LED_EXT
- LED_7 pad 2: unconnected-(LED_7-Pad2) -> LED_EXT
Routing:
- net LED_EXT: track 0.00 -> 151.4 mm, vias 0 -> 4
- net GND: track 446.0 -> 447.1 mm
- net DATA: track 205.2 -> 204.7 mm
Other:
- board text added: "+"
- board text added: "-"
- board text added: "DATA"
- board text added: "F4/A3"
- board text added: "F5/A2"
- board text added: "F6/A1"
- board text added: "LED"
- board text added: "Ver.1 Rev.3"
- board text added: "x"
- board text removed: "BAT"
- board text removed: "EXT1"
- board text removed: "EXT2"
- board text removed: "EXT3"
- board text removed: "GND DATA VCC"
- board text removed: "J1"
- board text removed: "Ver.1 Rev.2"
