File: pcb/ergotonic_f24-pcb-left/ergotonic_f24-pcb-left.kicad_sch (KiCad schematic)
At the start: 64 parts, among them J1 Conn_01x04, J3 Conn_01x06, SW1 SW_PUSH, SW10 SW_PUSH, SW11 SW_PUSH, SW12 SW_PUSH, SW13 SW_PUSH, SW14 SW_PUSH, SW15 SW_PUSH, SW16 SW_PUSH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

Commit message: Version 1 Revision 3
Connections:
- net LED_EXT: now reaches J3.6 (Pin_6)
- net LED_EXT: now also LED_7.2 (DOUT)
- no-connect marks 5 -> 3
Changed lines of the file:
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@@
   (junction (at 307.34 107.95) (diameter 0) (color 0 0 0 0)
   )
-  (no_connect (at 375.92 115.57))
   (no_connect (at 123.19 55.88))
   (no_connect (at 176.53 54.61))
-  (no_connect (at 171.45 69.85))
   (no_connect (at 38.1 22.86))
   (wire (pts (xy 157.48 132.08) (xy 185.42 132.08))
@@
     )
   )
+  (global_label "LED_EXT" (shape input) (at 375.92 115.57 0) (fields_autoplaced)
+    (effects (font (size 1.27 1.27)) (justify left))
+    (property "Intersheet References" "${INTERSHEET_REFS}" (id 0) (at 386.0741 115.4906 0)
+      (effects (font (size 1.27 1.27)) (justify left) hide)
+    )
+  )
   (global_label "RE1A" (shape input) (at 38.1 50.8 180) (fields_autoplaced)
     (effects (font (size 1.27 1.27)) (justify right))
@@
       (effects (font (size 1.27 1.27)) (justify left) hide)
     )
+  )
+  (global_label "LED_EXT" (shape input) (at 171.45 69.85 0) (fields_autoplaced)
+    (effects (font (size 1.27 1.27)) (justify left))
+    (property "Intersheet References" "${INTERSHEET_REFS}" (id 0) (at 181.6041 69.7706 0)
+      (effects (font (size 1.27 1.27)) (justify left) hide)
+    )
