File: pcb/ergotonic_f24-pcb-right/ergotonic_f24-pcb-right.kicad_pcb (KiCad board)
At the start: 2 copper layers, 167.2 x 112.2 mm, 66 parts, among them J2 Conn_01x04, J4 Conn_01x06, SW25 SW_PUSH, SW26 SW_PUSH, SW27 SW_PUSH, SW28 SW_PUSH, SW29 SW_PUSH, SW30 SW_PUSH, SW31 SW_PUSH, SW32 SW_PUSH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

Commit message: Version 1 Revision 3
Connections:
- J4 pad 6: unconnected-(J4-Pad6) -> LED_EXT2
- LED_15 pad 2: unconnected-(LED_15-Pad2) -> LED_EXT2
Routing:
- net LED_EXT2: track 0.00 -> 149.0 mm, vias 0 -> 2
- net GND2: track 625.7 -> 623.6 mm
- net ENC2_A: track 156.9 -> 156.0 mm
- net ENC2_B: track 149.1 -> 148.5 mm
Other:
- board text added: "+"
- board text added: "-"
- board text added: "DATA"
- board text added: "F4/A3"
- board text added: "F5/A2"
- board text added: "F6/A1"
- board text added: "LED"
- board text added: "Ver.1 Rev.3"
- board text added: "x"
- board text removed: "BAT"
- board text removed: "EXT2"
- board text removed: "EXT3"
- board text removed: "VCC DATA GND"
- board text removed: "Ver.1 Rev.2"
