File: pcb/ergotonic_f24-pcb-right/ergotonic_f24-pcb-right.kicad_sch (KiCad schematic)
At the start: 64 parts, among them J2 Conn_01x04, J4 Conn_01x06, SW25 SW_PUSH, SW26 SW_PUSH, SW27 SW_PUSH, SW28 SW_PUSH, SW29 SW_PUSH, SW30 SW_PUSH, SW31 SW_PUSH, SW32 SW_PUSH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

Commit message: Version 1 Revision 3
Connections:
- net LED_EXT2: now reaches J4.6 (Pin_6)
- net LED_EXT2: now also LED_15.2 (DOUT)
- no-connect marks 5 -> 3
Changed lines of the file:
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@@
   )
   (no_connect (at 254 27.94))
-  (no_connect (at 205.74 69.85))
   (no_connect (at 339.09 60.96))
-  (no_connect (at 382.27 203.2))
   (no_connect (at 200.66 54.61))
   (wire (pts (xy 175.26 223.52) (xy 175.26 242.57))
@@
       (effects (font (size 1.27 1.27)) (justify left) hide)
     )
+  )
+  (global_label "LED_EXT2" (shape input) (at 382.27 203.2 0) (fields_autoplaced)
+    (effects (font (size 1.27 1.27)) (justify left))
+    (property "Intersheet References" "${INTERSHEET_REFS}" (id 0) (at 393.6336 203.1206 0)
+      (effects (font (size 1.27 1.27)) (justify left) hide)
+    )
+  )
+  (global_label "LED_EXT2" (shape input) (at 205.74 69.85 0) (fields_autoplaced)
+    (effects (font (size 1.27 1.27)) (justify left))
+    (property "Intersheet References" "${INTERSHEET_REFS}" (id 0) (at 217.1036 69.7706 0)
+      (effects (font (size 1.27 1.27)) (justify left) hide)
+    )
